File: RS232-Relay/RS232-Relay.kicad_pcb (KiCad board)
At the start: 2 copper layers, 82.5 x 151 mm, 139 parts, among them J10 Relay 1-4, J11 Relay 1-4, J2 Conn_01x02, J4 Conn_01x09, J5 Conn_01x09, J7 RS232_1, J8 RS232_2, J9 Relay 1-4, K1 G5V-1, K13 G5V-1, K14 G5V-1, K15 G5V-1, K2 G5V-1, K3 G5V-1, K4 G5V-1, K5 G5V-1, K6 G5V-1, K7 G5V-1, K8 G5V-1, K9 G5V-1, Q1 2N3904, Q13 2N3904, Q14 2N3904, Q15 2N3904, Q2 2N3904, Q3 2N3904, Q4 2N3904, Q5 2N3904, Q6 2N3904, Q7 2N3904, Q8 2N3904, Q9 2N3904, SW2 SW_SPST, SW3 SW_SPST, U1 TEC2-1210WI, U2 LTV-847S, U3 PCF8575DBR, U4 MAX3232, U5 LTV-847S, U6 LTV-847S

Commit message: Figured out a solution, now for implementation
Parts:
- added JP10: Jumper_3_Bridged12, Jumper:SolderJumper-3_P1.3mm_Bridged2Bar12_RoundedPad1.0x1.5mm, F.Cu at (33.8, 89.6)
- added JP11: Jumper_3_Bridged12, Jumper:SolderJumper-3_P1.3mm_Bridged2Bar12_RoundedPad1.0x1.5mm, F.Cu at (45.5, 79.9)
- added JP12: Jumper_3_Bridged12, Jumper:SolderJumper-3_P1.3mm_Bridged2Bar12_RoundedPad1.0x1.5mm, F.Cu at (45.5, 99.2)
- added JP49: Jumper_3_Bridged12, Jumper:SolderJumper-3_P1.3mm_Bridged2Bar12_RoundedPad1.0x1.5mm, B.Cu at (102.7, 45.5)
- added JP5: Jumper_3_Bridged12, Jumper:SolderJumper-3_P1.3mm_Bridged2Bar12_RoundedPad1.0x1.5mm, F.Cu at (33.8, 79.9)
- added JP50: Jumper_3_Bridged12, Jumper:SolderJumper-3_P1.3mm_Bridged2Bar12_RoundedPad1.0x1.5mm, F.Cu at (22.1, 93.4)
- added JP51: Jumper_3_Bridged12, Jumper:SolderJumper-3_P1.3mm_Bridged2Bar12_RoundedPad1.0x1.5mm, F.Cu at (45.5, 112.8)
- added JP52: Jumper_3_Bridged12, Jumper:SolderJumper-3_P1.3mm_Bridged2Bar12_RoundedPad1.0x1.5mm, F.Cu at (22.1, 112.8)
- added JP53: Jumper_3_Bridged12, Jumper:SolderJumper-3_P1.3mm_Bridged2Bar12_RoundedPad1.0x1.5mm, F.Cu at (33.8, 83.7)
- added JP54: Jumper_3_Bridged12, Jumper:SolderJumper-3_P1.3mm_Bridged2Bar12_RoundedPad1.0x1.5mm, F.Cu at (33.8, 112.8)
- added JP55: Jumper_3_Bridged12, Jumper:SolderJumper-3_P1.3mm_Bridged2Bar12_RoundedPad1.0x1.5mm, F.Cu at (22.1, 103.1)
- added JP56: Jumper_3_Bridged12, Jumper:SolderJumper-3_P1.3mm_Bridged2Bar12_RoundedPad1.0x1.5mm, F.Cu at (18.0, 81.1)
- added JP57: Jumper_3_Bridged12, Jumper:SolderJumper-3_P1.3mm_Bridged2Bar12_RoundedPad1.0x1.5mm, F.Cu at (33.8, 103.1)
- added JP58: Jumper_3_Bridged12, Jumper:SolderJumper-3_P1.3mm_Bridged2Bar12_RoundedPad1.0x1.5mm, F.Cu at (33.8, 93.4)
- added JP59: Jumper_3_Bridged12, Jumper:SolderJumper-3_P1.3mm_Bridged2Bar12_RoundedPad1.0x1.5mm, F.Cu at (45.5, 83.7)
- added JP6: Jumper_3_Bridged12, Jumper:SolderJumper-3_P1.3mm_Bridged2Bar12_RoundedPad1.0x1.5mm, F.Cu at (33.8, 108.9)
- added JP60: Jumper_3_Bridged12, Jumper:SolderJumper-3_P1.3mm_Bridged2Bar12_RoundedPad1.0x1.5mm, F.Cu at (45.5, 103.1)
- added JP7: Jumper_3_Bridged12, Jumper:SolderJumper-3_P1.3mm_Bridged2Bar12_RoundedPad1.0x1.5mm, F.Cu at (22.1, 99.2)
- added JP8: Jumper_3_Bridged12, Jumper:SolderJumper-3_P1.3mm_Bridged2Bar12_RoundedPad1.0x1.5mm, F.Cu at (18.0, 77.2)
- added JP9: Jumper_3_Bridged12, Jumper:SolderJumper-3_P1.3mm_Bridged2Bar12_RoundedPad1.0x1.5mm, F.Cu at (33.8, 99.2)
- JP1: value Jumper_2_Bridged -> Jumper_3_Bridged12; footprint Jumper:SolderJumper-2_P1.3mm_Open_RoundedPad1.0x1.5mm -> Jumper:SolderJumper-3_P1.3mm_Bridged2Bar12_RoundedPad1.0x1.5mm; moved to B.Cu
- JP2, JP4: value Jumper_2_Open -> Jumper_3_Bridged12; footprint Jumper:SolderJumper-2_P1.3mm_Open_RoundedPad1.0x1.5mm -> Jumper:SolderJumper-3_P1.3mm_Bridged2Bar12_RoundedPad1.0x1.5mm
- JP3: value Jumper_2_Bridged -> Jumper_3_Bridged12; footprint Jumper:SolderJumper-2_P1.3mm_Open_RoundedPad1.0x1.5mm -> Jumper:SolderJumper-3_P1.3mm_Bridged2Bar12_RoundedPad1.0x1.5mm
- moved JP2 156.9 mm to (22.1, 89.6)
- moved JP1 156.6 mm to (102.7, 40.4), turned to -90 degrees
- moved JP4 148.8 mm to (22.1, 108.9)
- moved JP3 129.1 mm to (45.5, 108.9)
- moved R21 119.2 mm to (22.8, 76.7), turned to 0 degrees
- moved R48 111.4 mm to (27.0, 89.1), turned to 0 degrees
- moved R12 106.8 mm to (38.6, 79.4), turned to 0 degrees
- moved R3 98.3 mm to (27.0, 108.4), turned to 0 degrees
- moved R18 96.7 mm to (27.0, 98.7), turned to 0 degrees
- moved R30 96.2 mm to (50.3, 79.4), turned to 0 degrees
- moved R27 84.6 mm to (38.6, 89.1), turned to 0 degrees
- moved R24 84.4 mm to (38.6, 98.7), turned to 0 degrees
- moved R15 80.4 mm to (38.6, 108.4), turned to 0 degrees
- moved R33 74.9 mm to (50.3, 98.7), turned to 0 degrees
- moved R51 67.2 mm to (50.3, 108.4), turned to 0 degrees
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Connections:
- D1 pad 2: RELAY_ON -> +12V
- D10 pad 2: RELAY_ON -> +12V
- D11 pad 1: RELAY_ON -> +12V
- D12 pad 2: RELAY_ON -> +12V
- D13 pad 1: RELAY_ON -> +12V
- D14 pad 2: RELAY_ON -> +12V
- D15 pad 1: RELAY_ON -> +12V
- D16 pad 2: RELAY_ON -> +12V
- D17 pad 1: RELAY_ON -> +12V
- D18 pad 2: RELAY_ON -> +12V
- D19 pad 1: RELAY_ON -> +12V
- D2 pad 1: RELAY_ON -> +12V
- D20 pad 2: RELAY_ON -> +12V
- D21 pad 1: RELAY_ON -> +12V
- D28 pad 2: RELAY_ON -> +12V
- D29 pad 1: RELAY_ON -> +12V
- D3 pad 2: RELAY_ON -> +12V
- D30 pad 2: RELAY_ON -> +12V
- D31 pad 1: RELAY_ON -> +12V
- D32 pad 2: RELAY_ON -> +12V
- D33 pad 1: RELAY_ON -> +12V
- D4 pad 1: RELAY_ON -> +12V
- D8 pad 2: RELAY_ON -> +12V
- D9 pad 1: RELAY_ON -> +12V
- JP1 pad 1: GNDREF -> GND
- JP1 pad 2: RELAY_OFF -> /Relay-Module/Relay-NO-ISO/RELAY_OFF
- JP2 pad 1: +12V -> GND
- JP2 pad 2: RELAY_OFF -> /Relay-Module1/Relay-NO-ISO/RELAY_OFF
- JP3 pad 1: +12V -> GND
- JP3 pad 2: RELAY_ON -> /Relay-Module2/Relay-NO-ISO/RELAY_OFF
- JP4 pad 1: GNDREF -> GND
- JP4 pad 2: RELAY_ON -> /Relay-Module/Relay-NO-ISO1/RELAY_OFF
- K1 pad 1: RELAY_ON -> /Relay-Module/Relay-NO-ISO1/RELAY_OFF
- K1 pad 10: RELAY_ON -> /Relay-Module/Relay-NO-ISO1/RELAY_ON
- K1 pad 2: RELAY_ON -> +12V
- K13 pad 1: RELAY_ON -> /Relay-Module/Relay-NO-ISO/RELAY_OFF
- K13 pad 10: RELAY_ON -> /Relay-Module/Relay-NO-ISO/RELAY_ON
- K13 pad 2: RELAY_ON -> +12V
- K14 pad 1: RELAY_ON -> /Relay-Module1/Relay-NO-ISO/RELAY_OFF
- K14 pad 10: RELAY_ON -> /Relay-Module1/Relay-NO-ISO/RELAY_ON
- K14 pad 2: RELAY_ON -> +12V
- K15 pad 1: RELAY_ON -> /Relay-Module2/Relay-NO-ISO/RELAY_OFF
- K15 pad 10: RELAY_ON -> /Relay-Module2/Relay-NO-ISO/RELAY_ON
- K15 pad 2: RELAY_ON -> +12V
- K2 pad 1: RELAY_ON -> /Relay-Module1/Relay-NO-ISO1/RELAY_OFF
- K2 pad 10: RELAY_ON -> /Relay-Module1/Relay-NO-ISO1/RELAY_ON
- K2 pad 2: RELAY_ON -> +12V
- K3 pad 1: RELAY_ON -> /Relay-Module2/Relay-NO-ISO1/RELAY_OFF
- K3 pad 10: RELAY_ON -> /Relay-Module2/Relay-NO-ISO1/RELAY_ON
- K3 pad 2: RELAY_ON -> +12V
- K4 pad 1: RELAY_ON -> /Relay-Module/Relay-NO-ISO2/RELAY_OFF
- K4 pad 10: RELAY_ON -> /Relay-Module/Relay-NO-ISO2/RELAY_ON
- K4 pad 2: RELAY_ON -> +12V
- K5 pad 1: RELAY_ON -> /Relay-Module1/Relay-NO-ISO2/RELAY_OFF
- K5 pad 10: RELAY_ON -> /Relay-Module1/Relay-NO-ISO2/RELAY_ON
- K5 pad 2: RELAY_ON -> +12V
- K6 pad 1: RELAY_ON -> /Relay-Module2/Relay-NO-ISO2/RELAY_OFF
- K6 pad 10: RELAY_ON -> /Relay-Module2/Relay-NO-ISO2/RELAY_ON
- K6 pad 2: RELAY_ON -> +12V
- K7 pad 1: RELAY_ON -> /Relay-Module/Relay-NO-ISO3/RELAY_OFF
- K7 pad 10: RELAY_ON -> /Relay-Module/Relay-NO-ISO3/RELAY_ON
- K7 pad 2: RELAY_ON -> +12V
- K8 pad 1: RELAY_ON -> /Relay-Module1/Relay-NO-ISO3/RELAY_OFF
- K8 pad 10: RELAY_ON -> /Relay-Module1/Relay-NO-ISO3/RELAY_ON
- K8 pad 2: RELAY_ON -> +12V
- K9 pad 1: RELAY_ON -> /Relay-Module2/Relay-NO-ISO3/RELAY_OFF
- K9 pad 10: RELAY_ON -> /Relay-Module2/Relay-NO-ISO3/RELAY_ON
- K9 pad 2: RELAY_ON -> +12V
Routing:
- net RELAY_ON: track 370.1 -> 0.00 mm
- net +12V: track 47.7 -> 339.3 mm
- net GND: track 225.7 -> 263.9 mm
- net /Relay-Module1/Relay-NO-ISO3/OPTO_RIGHT_OUT: track 9.45 -> 0.00 mm
- net /Relay-Module2/Relay-NO-ISO3/OPTO_RIGHT_OUT: track 9.45 -> 0.11 mm
- net /Relay-Module/Relay-NO-ISO3/OPTO_RIGHT_OUT: track 9.45 -> 0.11 mm
- net /Relay-Module1/Relay-NO-ISO/OPTO_RIGHT_OUT: track 9.17 -> 0.00 mm
- net /Relay-Module2/Relay-NO-ISO/OPTO_RIGHT_OUT: track 9.17 -> 0.00 mm
- net /Relay-Module/Relay-NO-ISO/OPTO_RIGHT_OUT: track 9.17 -> 0.00 mm
- net /Relay-Module2/Relay-NO-ISO2/OPTO_RIGHT_OUT: track 5.02 -> 0.00 mm
- net /Relay-Module1/Relay-NO-ISO2/OPTO_RIGHT_OUT: track 5.02 -> 0.00 mm
- net /Relay-Module/Relay-NO-ISO2/OPTO_RIGHT_OUT: track 5.02 -> 0.00 mm
- net /Relay-Module2/Relay-NO-ISO1/OPTO_RIGHT_OUT: track 4.96 -> 0.00 mm
- net /Relay-Module1/Relay-NO-ISO1/OPTO_RIGHT_OUT: track 4.96 -> 0.00 mm
- net /Relay-Module/Relay-NO-ISO1/OPTO_RIGHT_OUT: track 4.96 -> 0.00 mm
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