File: RS232-Relay/RS232-Relay.kicad_pcb (KiCad board)
At the start: 2 copper layers, 82.5 x 151 mm, 159 parts, among them J10 Relay 1-4, J11 Relay 1-4, J2 Conn_01x02, J4 Conn_01x09, J5 Conn_01x09, J7 RS232_1, J8 RS232_2, J9 Relay 1-4, K1 G5V-1, K13 G5V-1, K14 G5V-1, K15 G5V-1, K2 G5V-1, K3 G5V-1, K4 G5V-1, K5 G5V-1, K6 G5V-1, K7 G5V-1, K8 G5V-1, K9 G5V-1, Q1 2N3904, Q13 2N3904, Q14 2N3904, Q15 2N3904, Q2 2N3904, Q3 2N3904, Q4 2N3904, Q5 2N3904, Q6 2N3904, Q7 2N3904, Q8 2N3904, Q9 2N3904, SW2 SW_SPST, SW3 SW_SPST, U1 TEC2-1210WI, U2 LTV-847S, U3 PCF8575DBR, U4 MAX3232, U5 LTV-847S, U6 LTV-847S

Commit message: Solution implemented
Parts:
- JP10, JP11, JP12, JP2, JP3, JP4, JP5, JP50, JP51, JP52, JP53, JP54, JP55, JP56, JP57, JP58, JP59, JP6, JP60, JP7, JP8, JP9: moved to B.Cu
- moved JP56 123.8 mm to (102.8, 171.4), turned to -90 degrees
- moved JP8 122.9 mm to (102.8, 166.3), turned to -90 degrees
- moved R21 119.2 mm to (115.8, 151.3), turned to 90 degrees
- moved JP59 113.4 mm to (102.8, 181.6), turned to -90 degrees
- moved JP11 112.3 mm to (102.8, 176.5), turned to -90 degrees
- moved R48 111.7 mm to (119.8, 151.3), turned to 90 degrees
- moved R12 107.0 mm to (117.8, 151.3), turned to 90 degrees
- moved JP53 103.6 mm to (102.7, 161.1), turned to -90 degrees
- moved JP5 102.7 mm to (102.7, 156.0), turned to -90 degrees
- moved JP4 99.6 mm to (102.7, 50.5), turned to -90 degrees
- moved JP50 99.0 mm to (102.7, 151.0), turned to -90 degrees
- moved JP52 98.8 mm to (102.7, 55.6), turned to -90 degrees
- moved R3 98.3 mm to (117.6, 70.2), turned to -90 degrees
- moved JP2 98.3 mm to (102.7, 145.9), turned to -90 degrees
- moved R18 96.7 mm to (119.4, 70.2), turned to -90 degrees
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Routing:
- net +12V: track 339.3 -> 575.2 mm
- net /Relay-Module2/Relay-NO-ISO3/OPTO_RIGHT_OUT: track 0.11 -> 9.82 mm
- net /Relay-Module1/Relay-NO-ISO3/OPTO_RIGHT_OUT: track 0.00 -> 9.55 mm
- net /Relay-Module/Relay-NO-ISO3/OPTO_RIGHT_OUT: track 0.11 -> 9.59 mm
- net /Relay-Module1/Relay-NO-ISO/OPTO_RIGHT_OUT: track 0.00 -> 9.17 mm
- net /Relay-Module2/Relay-NO-ISO/OPTO_RIGHT_OUT: track 0.00 -> 9.17 mm
- net /Relay-Module/Relay-NO-ISO/OPTO_RIGHT_OUT: track 0.00 -> 9.17 mm
- net /Relay-Module2/Relay-NO-ISO2/OPTO_RIGHT_OUT: track 0.00 -> 5.02 mm
- net /Relay-Module1/Relay-NO-ISO2/OPTO_RIGHT_OUT: track 0.00 -> 5.02 mm
- net /Relay-Module/Relay-NO-ISO2/OPTO_RIGHT_OUT: track 0.00 -> 5.02 mm
- net /Relay-Module2/Relay-NO-ISO1/OPTO_RIGHT_OUT: track 0.00 -> 4.96 mm
- net /Relay-Module1/Relay-NO-ISO1/OPTO_RIGHT_OUT: track 0.00 -> 4.96 mm
- net /Relay-Module/Relay-NO-ISO1/OPTO_RIGHT_OUT: track 0.00 -> 4.96 mm
- net GNDREF: track 32.0 -> 35.0 mm
- net /Relay-Module1/Relay-NO-ISO2/RELAY_OFF: track 0.00 -> 2.80 mm
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
Commit message: Schematic complete
Parts:
- added TP14: Backup, TestPoint:TestPoint_Pad_D1.0mm, B.Cu at (128.5, 124.0)
- added TP15: Backup, TestPoint:TestPoint_Pad_D1.0mm, B.Cu at (130.9, 102.9)
- added TP16: Backup, TestPoint:TestPoint_Pad_D1.0mm, B.Cu at (132.3, 125.2)
- added TP17: Backup, TestPoint:TestPoint_Pad_D1.0mm, B.Cu at (128.7, 122.0)
- added TP18: Backup, TestPoint:TestPoint_Pad_D1.0mm, B.Cu at (130.2, 100.9)
- added TP19: Backup, TestPoint:TestPoint_Pad_D1.0mm, B.Cu at (130.2, 125.6)
- added TP2: Backup, TestPoint:TestPoint_Pad_D1.0mm, B.Cu at (128.5, 102.0)
- added TP20: Backup, TestPoint:TestPoint_Pad_D1.0mm, B.Cu at (126.7, 122.3)
- added TP21: Backup, TestPoint:TestPoint_Pad_D1.0mm, B.Cu at (132.8, 102.1)
- added TP22: Backup, TestPoint:TestPoint_Pad_D1.0mm, B.Cu at (130.5, 123.6)
- added TP23: Backup, TestPoint:TestPoint_Pad_D1.0mm, B.Cu at (125.6, 117.1)
- added TP3: Backup, TestPoint:TestPoint_Pad_D1.0mm, B.Cu at (132.0, 127.2)
- moved G*** 35.1 mm to (115.8, 133.6)
Routing:
- net RELAY_IN_08: vias 0 -> 1
- net RELAY_IN_10: vias 0 -> 1
- net RELAY_IN_05: vias 0 -> 1
- net RELAY_IN_07: vias 0 -> 1
- net RELAY_IN_04: vias 0 -> 1
- net RELAY_IN_06: vias 0 -> 1
- net RELAY_IN_09: vias 0 -> 1
- net RELAY_IN_02: vias 0 -> 1
- net RELAY_IN_12: vias 0 -> 1
- net RELAY_IN_11: vias 0 -> 1
- net RELAY_IN_03: vias 0 -> 1
- net RELAY_IN_01: vias 0 -> 1
Other:
- outline, holes or cut-outs redrawn
- board text added: "12 channel 12V relay with RS232 control"
- board text added: "5V"
- board text added: "JLCJLCJLCJLC"

Commit message: Production v1
Parts:
- R10: value 50R -> 51R
- moved G*** 0.40 mm to (116.2, 133.6)
Routing:
- net RS232_1_TX: track 25.4 -> 24.7 mm
- net GNDREF: vias 94 -> 91
Other:
- board text added: "12 channel 12V relay with RS232 control v1.0"
- board text added: "Firmware Version:"
- board text removed: "12 channel 12V relay with RS232 control"
