File: RS232-Relay/RS232-Relay.kicad_sch (KiCad schematic)
At the start: 44 parts, among them J2 Conn_01x02, J4 Conn_01x09, J5 Conn_01x09, J7 RS232_1, J8 RS232_2, SW2 SW_SPST, SW3 SW_SPST, U1 TEC2-1210WI, U3 PCF8575DBR, U4 MAX3232

Commit message: Figuring out the relay NC/NO connections
Parts:
- added JP1, JP3: Jumper_2_Bridged, Jumper:SolderJumper-2_P1.3mm_Open_RoundedPad1.0x1.5mm, symbol Jumper:Jumper_2_Bridged
- added JP2, JP4: Jumper_2_Open, Jumper:SolderJumper-2_P1.3mm_Open_RoundedPad1.0x1.5mm, symbol Jumper:Jumper_2_Open
- added R9: 4K7, Resistor_SMD:R_0603_1608Metric, symbol Device:R_US
Connections:
- net +12V: now also JP2.1 (A), JP3.1 (A)
- net +3V3: now also R9.2
- net GNDREF: now also JP1.1 (A), JP4.1 (A)
- net I2C_INT: now also R9.1
- new net RELAY_OFF: JP1.2 (B), JP2.2 (B)
- new net RELAY_ON: JP3.2 (B), JP4.2 (B)

Commit message: Figured out a solution, now for implementation
Parts:
- removed JP1, JP3: Jumper_2_Bridged, Jumper:SolderJumper-2_P1.3mm_Open_RoundedPad1.0x1.5mm, symbol Jumper:Jumper_2_Bridged
- removed JP2, JP4: Jumper_2_Open, Jumper:SolderJumper-2_P1.3mm_Open_RoundedPad1.0x1.5mm, symbol Jumper:Jumper_2_Open

Commit message: 50Ohm -> 51Ohm resistor on LED
Parts:
- R10: value 50R -> 51R
Changed lines of the file:
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@@
 			)
 		)
-		(property "Value" "50R"
+		(property "Value" "51R"
 			(at 110.49 31.7499 0)
 			(effects

Commit message: Production v1
Parts:
- U3: LCSC (none) -> C2863388
Changed lines of the file:
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@@
+			)
+		)
+		(property "LCSC" "C2863388"
+			(at 351.79 68.58 0)
+			(effects
+				(font
+					(size 1.27 1.27)
+				)
+				(hide yes)
 			)
 		)
